File: cm4_gpio.kicad_sch (KiCad schematic)
At the start: 14 parts, among them J4 ARJM11B1-502-AB-EW2, U2 TPD4EUSB30, U3 TPD4EUSB30, U4 74LVC1G07SE-7

Commit message: Prep Rev2
Parts:
- removed JP1: Enable USB Boot, Connector_PinHeader_1.27mm:PinHeader_1x02_P1.27mm_Vertical, symbol Jumper:Jumper_2_Open
- removed U4: 74LVC1G07SE-7, Package_TO_SOT_SMD:SOT-353_SC-70-5, symbol CM4IO:74LVC1G07_copy
- added C1, C3: 1uF, Capacitor_SMD:C_0402_1005Metric, symbol Device:C
- added C52: 1uF, Capacitor_SMD:C_1206_3216Metric, symbol Device:C
- added J7: ~, Connector_PinHeader_2.54mm:PinHeader_1x04_P2.54mm_Vertical_SMD_Pin1Left, symbol Connector_Generic:Conn_01x04
- added R33, R34: 4.7k, Resistor_SMD:R_0402_1005Metric, symbol Device:R
- added SW1: SW_DIP_x05, Button_Switch_SMD:SW_DIP_SPSTx05_Slide_KingTek_DSHP05TJ_W5.25mm_P1.27mm_JPin, symbol Switch:SW_DIP_x05
- added TP1, TP3, TP4, TP5: TestPoint, TestPoint:TestPoint_Keystone_5000-5004_Miniature, symbol Connector:TestPoint
- added U1: SN74LVC1G11, Package_SON:Texas_USON-6_1x1.45mm_P0.5mm_SMD, symbol 74xGxx:74LVC1G11
- added U12: 24LC32, Package_SO:SOIC-8_3.9x4.9mm_P1.27mm, symbol Memory_EEPROM:24LC32
- added U4: 74LVC1G07, Package_SON:Texas_USON-6_1x1.45mm_P0.5mm_SMD, symbol 74xGxx:74LVC1G07
- R1: renamed from R8; footprint Resistor_SMD:R_0603_1608Metric_Pad0.98x0.95mm_HandSolder -> Resistor_SMD:R_0402_1005Metric
- R4: renamed from R9; footprint Resistor_SMD:R_0603_1608Metric_Pad0.98x0.95mm_HandSolder -> Resistor_SMD:R_0402_1005Metric
- renumbered C12 to C2, J4 to J1, R1 to R2, R2 to R3, TP1 to TP2
Connections:
- net +3.3V: now also C3.1, C52.1, J7.1 (Pin_1), R33.2, R34.2, U12.8 (VCC), U4.6 (VCC)
- net +5V: now also C1.1, U1.5 (VCC)
- net GND: now also C1.2, C3.2, C52.2, J7.4 (Pin_4), SW1.10, SW1.6, SW1.7, SW1.8, SW1.9, U1.2 (GND), U12.4 (GND), U4.3 (GND)
- net TRD1_N: now also J1.3 (TD2+); no longer J1.4 (TD2-)
- net TRD1_P: now also J1.4 (TD2-); no longer J1.3 (TD2+)
- net TRD3_N: now also J1.9 (TD4+); no longer J1.10 (TD4-)
- net TRD3_P: now also J1.10 (TD4-); no longer J1.9 (TD4+)
- net nEXTRST: now also TP1.1
- net nPWR_LED: now also U4.2
- net at R4.2: now also U4.4
- net at Module1.93 (nRPIBOOT): now also SW1.3
- net EEPROM_nWP: now reaches Module1.20 (EEPROM_nWP)
- net EEPROM_nWP: now also SW1.5
- net UART.RX: now reaches Module1.28 (GPIO13)
- net UART.RX: now also TP4.1
- net Wireless.SWDIO: now reaches Module1.30 (GPIO6)
- net UART.TX: now reaches Module1.31 (GPIO12)
- net UART.TX: now also TP5.1
- net ID_SC: now reaches Module1.35 (ID_SC)
- net ID_SC: now also J7.3 (Pin_3), U12.6 (SCL)
- net ID_SD: now reaches Module1.36 (ID_SD)
- net ID_SD: now also J7.2 (Pin_2), U12.5 (SDA)
- net Wireless.SWCLK: now reaches Module1.37 (GPIO7)
- net Wireless.~{RESET}: now reaches Module1.41 (GPIO25)
- net Wireless.~{BOOT}: now reaches Module1.45 (GPIO24)
- net I2C.SDA: now reaches Module1.46 (GPIO22)
- net I2C.SDA: now also R33.1
- net I2C.SCL: now reaches Module1.47 (GPIO23)
- net I2C.SCL: now also R34.1
- net +1V8: now reaches Module1.88 (+1.8v_(Output))
- net +1V8: now also Module1.90 (+1.8v_(Output))
- net at Module1.89 (WiFi_nDisable): now also SW1.1
- net at Module1.91 (BT_nDisable): now also SW1.2
- net RUN_PG: now reaches Module1.92 (RUN_PG)
- net RUN_PG: now also TP3.1
- net at Module1.99 (Global_EN): now also U1.4
- net SPI0_CE0 renamed Wireless.TXD
- net SPI0_CE1: no longer names the net of Module1.82 (SDA0)
- net SPI0_MISO renamed Wireless.RXD
- net SPI0_MOSI renamed Wireless.CTS
- net SPI0_SCLK renamed Wireless.RTS
- net UART_WIRELESS_CTS: no longer names the net of Module1.29 (GPIO16)
- net UART_WIRELESS_RTS: no longer names the net of Module1.50 (GPIO17)
- net UART_WIRELESS_RX: no longer names the net of Module1.51 (GPIO15)
- net UART_WIRELESS_TX: no longer names the net of Module1.55 (GPIO14)
- new net: SW1.4, U1.6
- new net 3V3_PG: U1.1
- new net 5V_PG: U1.3
- no-connect marks 0 -> 4
Other:
- moved on the sheet: Module1A, R2, R3, TP2, U2, U3

Commit message: Rev 2
Parts:
- C40: renamed from C1; footprint Capacitor_SMD:C_0402_1005Metric -> Capacitor_SMD:C_0603_1608Metric
- C43: renamed from C52; footprint Capacitor_SMD:C_1206_3216Metric -> Capacitor_SMD:C_0402_1005Metric
- U11: renamed from U12; LCSC Part # (none) -> C615215; MPN (none) -> 24LC32A/SN
- U13: renamed from U2; LCSC Part # (none) -> C90627
- U14: renamed from U3; LCSC Part # (none) -> C90627
- U2: renamed from U4; LCSC Part # (none) -> C2675513; MPN (none) -> SN74LVC1G07DRY
- U9: renamed from U1; MPN (none) -> SN74LVC1G11DRYR
- renumbered C3 to C14, C2 to C49, J7 to J4, J1 to J5, R4 to R2, R34 to R28, R33 to R29, R2 to R38, R3 to R39, TP4 to TP10, TP5 to TP11, TP1 to TP12, TP2 to TP16, TP3 to TP9
Connections:
- net TRD3_N: now also J5.10 (TD4-), U13.1 (D1+), U13.10; no longer J5.9 (TD4+), U13.2 (D1-), U13.9
- net TRD3_P: now also J5.9 (TD4+), U13.2 (D1-), U13.9; no longer J5.10 (TD4-), U13.1 (D1+), U13.10
