File: cm4_highspeed.kicad_sch (KiCad schematic)
At the start: 4 parts, among them J2 Bus_M.2_Socket_M

Commit message: Prep Rev2
Parts:
- added C4, C5, C56, C6: 1uF, Capacitor_SMD:C_0402_1005Metric, symbol Device:C
- added D3: Orange 1.9V 5mA, LED_SMD:LED_0603_1608Metric, symbol Device:LED
- added Q1: DMG1012T, Package_TO_SOT_SMD:SOT-523, symbol Transistor_FET:DMG1012T
- added R5: 10k, Resistor_SMD:R_0603_1608Metric, symbol Device:R
- added R6: 1k, Resistor_SMD:R_0402_1005Metric, symbol Device:R
- added U5: SN74LVC1G3157, Package_TO_SOT_SMD:SOT-363_SC-70-6, symbol 74xGxx:74LVC1G3157
- H5, H6: footprint MountingHole:MountingHole_3.7mm_Pad -> MountingHole:MountingHole_3.7mm_Pad_TopOnly; MPN KFS2-M2 -> 9774015151R
Connections:
- net +3V3: now also C4.1, C5.1, C56.1, C6.1, D3.2 (A), R5.1, U5.5 (VCC)
- net GND: now also C4.2, C5.2, C56.2, C6.2, U5.2 (GND)
- net PCIE_CLK_N: now also Module1.110 (PCIe_CLK_P); no longer Module1.112 (PCIe_CLK_N)
- net PCIE_CLK_P: now also Module1.112 (PCIe_CLK_N); no longer Module1.110 (PCIe_CLK_P)
- net PCIE_CLK_nREQ: now also U5.3; no longer J2.52 (~{CLKREQ})
- net PCIE_RX_N: now also Module1.116 (PCIe_RX_P); no longer Module1.118 (PCIe_RX_N)
- net PCIE_RX_P: now also Module1.118 (PCIe_RX_N); no longer Module1.116 (PCIe_RX_P)
- net PCIE_TX_N: now also Module1.122 (PCIe_TX_P); no longer Module1.124 (PCIe_TX_N)
- net PCIE_TX_P: now also Module1.124 (PCIe_TX_N); no longer Module1.122 (PCIe_TX_P)
- net PCIE_nRST: now also Q1.3 (D); no longer J2.50 (~{PERST})
- net at J2.10 (DAS/~{DSS}/~{LED1}): now also R6.1
- new net: D3.1 (K), R6.2
- new net: J2.50 (~{PERST}), Q1.2 (S)
- new net: J2.52 (~{CLKREQ}), U5.4
- new net: R5.2, U5.1
- new net 3V3_PG: Q1.1 (G), U5.6
- no-connect marks 17 -> 16
Other:
- note added: "Swapped polarities for easier routing"
- title: (none) -> M.2 socket
- moved on the sheet: H5, H6, J2, Module1B

Commit message: Rev 2
Parts:
- D3: LCSC Part # (none) -> C18198804
- J3: renamed from J2; LCSC Part # (none) -> C4527433
- Q1: LCSC Part # (none) -> C42412320; MPN (none) -> DMG1012T-13
- U10: renamed from U5; LCSC Part # (none) -> C2870968; MPN (none) -> SN74LVC1G3157DRYR
- renumbered C6 to C35, C5 to C38, C4 to C39, C56 to C41, H6 to H3, H5 to H4, R6 to R3, R5 to R30
Changed lines of the file:
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@@
 		(dnp no)
 		(fields_autoplaced yes)
-		(property "Reference" "R6"
+		(property "Reference" "R3"
 			(at 245.11 74.93 0)
 			(effects
@@
 			(project "rpi-cm-ssd"
 				(path "/d596c5fc-bc79-4446-9328-b82e41a34e97/f931d0e3-8690-4710-a3ba-0dade8097dcb"
-					(reference "R6")
+					(reference "R3")
 					(unit 1)
 				)
@@
 		(dnp no)
 		(fields_autoplaced yes)
-		(property "Reference" "C5"
+		(property "Reference" "C38"
 			(at 260.35 29.2099 0)
 			(effects
@@
 			(project ""
 				(path "/d596c5fc-bc79-4446-9328-b82e41a34e97/f931d0e3-8690-4710-a3ba-0dade8097dcb"
-					(reference "C5")
+					(reference "C38")
 					(unit 1)
 				)
@@
 		)
 		(property "MPN" "HSMD-C190"
+			(at 242.57 67.31 90)
+			(effects
+				(font
+					(size 1.27 1.27)
+				)
+				(hide yes)
+			)
+		)
+		(property "LCSC Part #" "C18198804"
 			(at 242.57 67.31 90)
 			(effects
@@
 			)
 		)
+		(property "LCSC Part #" "C42412320"
+			(at 152.4 34.29 90)
+			(effects
+				(font
+					(size 1.27 1.27)
+				)
+				(hide yes)
+			)
+		)
+		(property "MPN" "DMG1012T-13"
+			(at 152.4 34.29 90)
+			(effects
+				(font
+					(size 1.27 1.27)
+				)
+				(hide yes)
+			)
+		)
 		(pin "1"
 		)
@@
 		(dnp no)
 		(fields_autoplaced yes)
-		(property "Reference" "J2"
+		(property "Reference" "J3"
 			(at 212.8394 29.21 0)
 			(effects
@@
 			)
 		)
+		(property "LCSC Part #" "C4527433"
+			(at 210.82 80.01 0)
+			(effects
+				(font
+					(size 1.27 1.27)
+				)
+				(hide yes)
+			)
+		)
 		(pin "1"
 		)
@@
 			(project "rpi-cm-ssd"
 				(path "/d596c5fc-bc79-4446-9328-b82e41a34e97/f931d0e3-8690-4710-a3ba-0dade8097dcb"
-					(reference "J2")
+					(reference "J3")
 					(unit 1)
 				)
@@
 		(dnp no)
 		(fields_autoplaced yes)
-		(property "Reference" "C4"
+		(property "Reference" "C39"
 			(at 247.65 29.2099 0)
 			(effects
@@
 			(project ""
 				(path "/d596c5fc-bc79-4446-9328-b82e41a34e97/f931d0e3-8690-4710-a3ba-0dade8097dcb"
-					(reference "C4")
+					(reference "C39")
 					(unit 1)
 				)
@@
 		(on_board yes)
 		(dnp no)
-		(property "Reference" "U5"
+		(property "Reference" "U10"
 			(at 153.67 57.15 0)
 			(effects
@@
 			)
 		)
+		(property "MPN" "SN74LVC1G3157DRYR"
+			(at 152.4 69.85 0)
+			(effects
+				(font
+					(size 1.27 1.27)
+				)
+				(hide yes)
+			)
+		)
+		(property "LCSC Part #" "C2870968"
+			(at 152.4 69.85 0)
+			(effects
+				(font
+					(size 1.27 1.27)
+				)
+				(hide yes)
+			)
+		)
 		(pin "5"
 		)
@@
 			(project "rpi-cm-ssd"
 				(path "/d596c5fc-bc79-4446-9328-b82e41a34e97/f931d0e3-8690-4710-a3ba-0dade8097dcb"
-					(reference "U5")
+					(reference "U10")
 					(unit 1)
 				)
@@
 		(dnp no)
 		(fields_autoplaced yes)
-		(property "Reference" "C56"
+		(property "Reference" "C41"
 			(at 134.62 96.5199 0)
 			(effects
@@
 			(project ""
 				(path "/d596c5fc-bc79-4446-9328-b82e41a34e97/f931d0e3-8690-4710-a3ba-0dade8097dcb"
-					(reference "C56")
+					(reference "C41")
 					(unit 1)
 				)
@@
 		(dnp no)
 		(fields_autoplaced yes)
-		(property "Reference" "H5"
+		(property "Reference" "H4"
 			(at 198.12 149.8599 0)
 			(effects
@@
 			(project "rpi-cm-ssd"
 				(path "/d596c5fc-bc79-4446-9328-b82e41a34e97/f931d0e3-8690-4710-a3ba-0dade8097dcb"
-					(reference "H5")
+					(reference "H4")
 					(unit 1)
 				)
@@
 		(dnp no)
 		(fields_autoplaced yes)
-		(property "Reference" "R5"
+		(property "Reference" "R30"
 			(at 134.62 58.42 90)
 			(effects
@@
 			(project "rpi-cm-ssd"
 				(path "/d596c5fc-bc79-4446-9328-b82e41a34e97/f931d0e3-8690-4710-a3ba-0dade8097dcb"
-					(reference "R5")
+					(reference "R30")
 					(unit 1)
 				)
@@
 		(dnp no)
 		(fields_autoplaced yes)
-		(property "Reference" "U5"
+		(property "Reference" "U10"
 			(at 152.4 83.82 90)
 			(effects
@@
 			)
 		)
+		(property "MPN" "SN74LVC1G3157DRYR"
+			(at 152.4 91.44 0)
+			(effects
+				(font
+					(size 1.27 1.27)
+				)
+				(hide yes)
+			)
+		)
+		(property "LCSC Part #" "C2870968"
+			(at 152.4 91.44 0)
+			(effects
+				(font
+					(size 1.27 1.27)
+				)
+				(hide yes)
+			)
+		)
 		(pin "5"
 		)
@@
 			(project "rpi-cm-ssd"
 				(path "/d596c5fc-bc79-4446-9328-b82e41a34e97/f931d0e3-8690-4710-a3ba-0dade8097dcb"
-					(reference "U5")
+					(reference "U10")
 					(unit 2)
 				)
@@
 		(dnp no)
 		(fields_autoplaced yes)
-		(property "Reference" "H6"
+		(property "Reference" "H3"
 			(at 220.98 149.8599 0)
 			(effects
@@
 			(project "rpi-cm-ssd"
 				(path "/d596c5fc-bc79-4446-9328-b82e41a34e97/f931d0e3-8690-4710-a3ba-0dade8097dcb"
-					(reference "H6")
+					(reference "H3")
 					(unit 1)
 				)
@@
 		(dnp no)
 		(fields_autoplaced yes)
-		(property "Reference" "C6"
+		(property "Reference" "C35"
 			(at 273.05 29.2099 0)
 			(effects
@@
 			(project ""
 				(path "/d596c5fc-bc79-4446-9328-b82e41a34e97/f931d0e3-8690-4710-a3ba-0dade8097dcb"
-					(reference "C6")
+					(reference "C35")
 					(unit 1)
 				)
