File: power.kicad_sch (KiCad schematic)
At the start: 66 parts, among them J1 USB_C_Receptacle, J3 PD controller EEPROM programm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, U1 TVS2200DRV, U10 TPS65283-1RGER, U5 CAT24C256, U6 TPS25750DRJKT, U7 PAC1951-1

Commit message: Prep Rev2
Parts:
- removed U1: TVS2200DRV, Package_SON:WSON-6-1EP_2x2mm_P0.65mm_EP1x1.6mm, symbol Power_Protection:TVS2200DRV
- added C39: 100uF, Capacitor_Tantalum_SMD:CP_EIA-3216-10_Kemet-I, symbol Device:C_Polarized
- added R15: 100k, Resistor_SMD:R_0402_1005Metric, symbol Device:R
- added TP10, TP11: TestPoint, TestPoint:TestPoint_Keystone_5000-5004_Miniature, symbol Connector:TestPoint
- added U7: TVS2200DRV, Package_SON:WSON-6-1EP_2x2mm_P0.65mm_EP1x1.6mm, symbol Power_Protection:TVS2200DRV
- C16: renamed from C33; value 22uF -> 47uF
- C18: renamed from C35; value 22uF -> 47uF
- C22: renamed from C34; footprint Capacitor_SMD:C_0402_1005Metric -> Capacitor_SMD:C_1206_3216Metric
- C7: renamed from C13; value 0.1uF -> 1uF
- J4: renamed from J3; footprint Connector_PinHeader_2.54mm:PinHeader_1x04_P2.54mm_Vertical -> Connector_PinHeader_2.54mm:PinHeader_1x04_P2.54mm_Vertical_SMD_Pin1Left
- R22: renamed from R25; value 17k -> 40.2k
- R23: renamed from R26; value 100k -> 75k
- TP13: renamed from TP4; footprint TestPoint:TestPoint_Pad_D1.0mm -> TestPoint:TestPoint_Keystone_5000-5004_Miniature
- TP9: renamed from TP6; footprint TestPoint:TestPoint_Pad_D1.0mm -> TestPoint:TestPoint_Keystone_5000-5004_Miniature
- renumbered C14 to C10, C15 to C11, C3 to C12, C4 to C13, C25 to C14, C5 to C15, C6 to C17, C31 to C19, C32 to C20, C37 to C21, C36 to C23, C39 to C24, C40 to C25, C38 to C26, C41 to C27, C16 to C28, C17 to C29, C18 to C30, C23 to C31, C44 to C32, C45 to C33, C7 to C34, C46 to C35, C24 to C36, C47 to C37, C48 to C38, C1 to C8, C2 to C9, J1 to J3, L2 to L1, L3 to L2, R16 to R10, R17 to R11, R18 to R12, R3 to R13, R4 to R14, R19 to R16, R20 to R17, R21 to R18, R22 to R19, R23 to R20, R24 to R21, R27 to R24, R28 to R25, R10 to R26, R29 to R27, R5 to R7, R6 to R8, R7 to R9, TP2 to TP12, TP5 to TP14, TP3 to TP8, U5 to U6, U6 to U8, U7 to U9
Connections:
- net +3.3V: now also R15.1
- net +5V: now also C39.1
- net GND: now also U8.10 (I2Cs_IRQ_N), U8.13 (GPIO11), U8.19 (GPIO3), U8.26 (GPIO4_USB_P), U8.27 (GPIO5_USB_N), U8.36 (GPIO7), U8.37 (GPIO6), U8.5 (GPIO0), U8.6 (GPIO1), U8.7 (GPIO2), C39.2, U7.1 (GND), U7.2 (GND), U7.3 (GND), U7.7 (GND)
- net ~{PWRDN}: now also R15.2
- net VIN: now reaches J3.A4 (VBUS), J3.A9 (VBUS), J3.B4 (VBUS), J3.B9 (VBUS), R13.1
- net VIN: now also U7.4 (IN), U7.5 (IN), U7.6 (IN)
- net CURRENT_SENSE_P: now reaches R13.2, U9.11 (IN1+)
- net CURRENT_SENSE_N: now reaches R13.3, U9.12 (IN1-)
- net I2C_SCL renamed I2C.SCL
- net I2C_SDA renamed I2C.SDA
- net PGOOD1 renamed 3V3_PG
- net 3V3_PG: now also TP10.1
- net PGOOD2 renamed 5V_PG
- net 5V_PG: now also TP11.1
- no-connect marks 25 -> 15
Other:
- note added: "7-bit I²C address as target device is 0100000 (0x20)"
- note added: "7-bit I²C address is 1010000 (0x50)"
- note added: "USB ESD protection"
- moved on the sheet: C15, C17, J4, R13, R14, TP12, TP13, TP14, TP8, TP9, U9

Commit message: Rev 2
Parts:
- removed C12, C13: 10nF, Capacitor_SMD:C_0402_1005Metric, symbol Device:C
- added C5, C6: 10nF, Capacitor_SMD:C_0402_1005Metric, symbol Device:C
- added R20: 100k, Resistor_SMD:R_0402_1005Metric, symbol Device:R
- J1: renamed from J3; LCSC Part # (none) -> C5119948
- L1: renamed from L2; LCSC Part # (none) -> C3040367
- L2: renamed from L1; LCSC Part # (none) -> C3040367
- R21: renamed from R15; footprint Resistor_SMD:R_0402_1005Metric -> Resistor_SMD:R_0805_2012Metric
- U1: renamed from U6; LCSC Part # (none) -> C36533643
- U4: renamed from U7; LCSC Part # (none) -> C523793
- U5: renamed from U10; LCSC Part # (none) -> C2071487
- U6: renamed from U9; LCSC Part # (none) -> C5226663
- U7: renamed from U8; LCSC Part # (none) -> C2868209
- renumbered C7 to C1, C39 to C10, C31 to C11, C32 to C12, C28 to C13, C33 to C16, C25 to C17, C37 to C18, C10 to C19, C30 to C2, C11 to C20, C35 to C21, C17 to C22, C15 to C23, C21 to C24, C36 to C25, C34 to C27, C24 to C28, C22 to C29, C27 to C3, C19 to C30, C20 to C31, C23 to C32, C14 to C33, C18 to C36, C16 to C37, C29 to C4, C38 to C7, J4 to J2, R25 to R10, R24 to R11, R22 to R12, R17 to R13, R21 to R14, R20 to R15, R11 to R16, R10 to R17, R14 to R18, R13 to R19, R26 to R22, R19 to R24, R18 to R25, R16 to R26, R7 to R5, R27 to R6, R8 to R7, R12 to R8, TP11 to TP1, TP9 to TP15, TP14 to TP4, TP13 to TP5, TP10 to TP6, TP8 to TP7, TP12 to TP8
Connections:
- net +3.3V: now also R20.1
- net GND: now also C5.2, C6.2
- net METER_ALERT: now also R20.2
- net VBUS: no longer C8.1, C9.1
- net VIN: now also C8.1, C9.1, C5.1, C6.1
Other:
- moved on the sheet: C33, R21, U4
