File: rpi-cm-ssd.kicad_pcb (KiCad board)
At the start: 4 copper layers, 87.3 x 55.1 mm, 127 parts, among them J1 USB_C_Receptacle, J2 Bus_M.2_Socket_M, J3 PD controller EEPROM programm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, J4 ARJM11B1-502-AB-EW2, J5 690-008-221-904, U1 TVS2200DRV, U10 TPS65283-1RGER, U11 TCN75AVUA, U12 TCN75AVUA, U13 MGM210PB32JIA2, U2 TPD4EUSB30, U3 TPD4EUSB30, U4 74LVC1G07SE-7, U5 CAT24C256, U6 TPS25750DRJKT, U7 PAC1951-1, U8 USB2512, U9 SC18IS604PWJ, Y1 24MHz

Commit message: Prep Rev2
Parts:
- removed AE1: A-4JA, A-4JA:A-4JA
- removed the C10 at (105.1, 79.0)
- removed the C33 at (105.6, 53.4)
- removed JP1: Enable USB Boot, Connector_PinHeader_1.27mm:PinHeader_1x02_P1.27mm_Vertical
- removed the R13 at (114.2, 81.8)
- removed the R14 at (115.2, 80.0)
- removed REF**: Symbol_GNU-Logo_SilkscreenTop, Symbol:Symbol_GNU-Logo_SilkscreenTop
- removed REF**: OSHW-Symbol_6.7x6mm_SilkScreen, Symbol:OSHW-Symbol_6.7x6mm_SilkScreen
- removed REF**: KiCad-Logo2_5mm_SilkScreen, Symbol:KiCad-Logo2_5mm_SilkScreen
- removed the TP12 at (95.8, 84.0)
- removed TP7: TestPoint, TestPoint:TestPoint_THTPad_D2.0mm_Drill1.0mm
- removed the TP8 at (76.7, 84.0)
- removed the TP9 at (89.6, 84.0)
- removed the U9 at (109.7, 78.9)
- added C1: 1uF, Capacitor_SMD:C_0402_1005Metric, F.Cu at (141.2, 48.0)
- added C16: 47uF, Capacitor_SMD:C_0805_2012Metric, F.Cu at (86.1, 43.2)
- added C3: 1uF, Capacitor_SMD:C_0402_1005Metric, F.Cu at (76.7, 33.2)
- added C39: 100uF, Capacitor_Tantalum_SMD:CP_EIA-3216-10_Kemet-I, F.Cu at (150.0, 57.6)
- added C4: 1uF, Capacitor_SMD:C_0402_1005Metric, F.Cu at (78.1, 42.4)
- added C40: 100uF, Capacitor_Tantalum_SMD:CP_EIA-3216-10_Kemet-I, F.Cu at (68.2, 57.1)
- added C42: 10uF, Capacitor_SMD:C_0603_1608Metric, F.Cu at (66.0, 57.6)
- added C44: 10uF, Capacitor_SMD:C_0603_1608Metric, F.Cu at (80.0, 54.3)
- added C45: 10uF, Capacitor_SMD:C_0603_1608Metric, F.Cu at (81.5, 55.4)
- added C5: 1uF, Capacitor_SMD:C_0402_1005Metric, F.Cu at (78.1, 41.4)
- added C52: 1uF, Capacitor_SMD:C_1206_3216Metric, B.Cu at (125.0, 58.8)
- added C55: 1uF, Capacitor_SMD:C_0402_1005Metric, F.Cu at (75.7, 37.0)
- added C56: 1uF, Capacitor_SMD:C_0402_1005Metric, F.Cu at (90.5, 45.9)
- added C6: 1uF, Capacitor_SMD:C_0402_1005Metric, F.Cu at (98.2, 42.7)
- added D3: Orange 1.9V 5mA, LED_SMD:LED_0603_1608Metric, F.Cu at (65.0, 33.8)
- added D4: Blue 2.8V @ 5mA, LED_SMD:LED_0603_1608Metric, F.Cu at (66.6, 33.8)
- added J6: CONUFL001-SMD-T, Connector_Coaxial:U.FL_Hirose_U.FL-R-SMT-1_Vertical, B.Cu at (112.3, 34.2)
- added J7: ~, Connector_PinHeader_2.54mm:PinHeader_1x04_P2.54mm_Vertical_SMD_Pin1Left, B.Cu at (116.9, 58.6)
- added Q1: DMG1012T, Package_TO_SOT_SMD:SOT-523, F.Cu at (90.8, 43.3)
- added R33: 4.7k, Resistor_SMD:R_0402_1005Metric, F.Cu at (147.4, 14.3)
- added R34: 4.7k, Resistor_SMD:R_0402_1005Metric, F.Cu at (147.4, 16.3)
- added R37: 1k, Resistor_SMD:R_0402_1005Metric, F.Cu at (73.1, 35.7)
- added R38: 1k, Resistor_SMD:R_0603_1608Metric, B.Cu at (132.1, 34.2)
- added R39: 10k, Resistor_SMD:R_0603_1608Metric, B.Cu at (132.1, 35.7)
- added R40: 10k, Resistor_SMD:R_0603_1608Metric, B.Cu at (113.5, 38.5)
- added R5: 10k, Resistor_SMD:R_0603_1608Metric, F.Cu at (89.0, 46.0)
- added R6: 1k, Resistor_SMD:R_0402_1005Metric, F.Cu at (73.1, 36.7)
- added SW1: SW_DIP_x05, Button_Switch_SMD:SW_DIP_SPSTx05_Slide_KingTek_DSHP05TJ_W5.25mm_P1.27mm_JPin, B.Cu at (141.0, 42.8)
- added TP1: TestPoint, TestPoint:TestPoint_Keystone_5000-5004_Miniature, B.Cu at (113.0, 45.4)
- added TP13: TestPoint, TestPoint:TestPoint_Keystone_5000-5004_Miniature, F.Cu at (149.8, 81.3)
- added TP15: TestPoint, TestPoint:TestPoint_Keystone_5000-5004_Miniature, B.Cu at (76.4, 60.5)
- added TP16: TestPoint, TestPoint:TestPoint_Keystone_5000-5004_Miniature, B.Cu at (75.7, 56.3)
- added TP18: TestPoint, TestPoint:TestPoint_Keystone_5000-5004_Miniature, B.Cu at (156.6, 58.5)
- added TP20: TestPoint, TestPoint:TestPoint_Keystone_5000-5004_Miniature, B.Cu at (153.4, 54.1)
- added TP3: TestPoint, TestPoint:TestPoint_Keystone_5000-5004_Miniature, B.Cu at (130.8, 46.6)
- added TP5: TestPoint, TestPoint:TestPoint_Keystone_5000-5004_Miniature, F.Cu at (144.6, 80.2)
- added U12: 24LC32, Package_SO:SOIC-8_3.9x4.9mm_P1.27mm, B.Cu at (130.0, 59.2)
- added U15: SN74LVC1G07, Package_SON:Texas_USON-6_1x1.45mm_P0.5mm_SMD, F.Cu at (75.1, 35.8)
- added U5: SN74LVC1G3157, Package_TO_SOT_SMD:SOT-363_SC-70-6, F.Cu at (92.4, 46.1)
- added U7: TVS2200DRV, Package_SON:WSON-6-1EP_2x2mm_P0.65mm_EP1x1.6mm, F.Cu at (152.9, 38.4)
- C18: renamed from C35; value 22uF -> 47uF
- C2: renamed from C12; moved to F.Cu
- C22: renamed from C34; footprint Capacitor_SMD:C_0402_1005Metric -> Capacitor_SMD:C_1206_3216Metric
- C41: renamed from C8; value 15pF -> 15pF C0G
- C43: renamed from C9; value 15pF -> 15pF C0G
- C53: renamed from C11; value 0.1uF -> 1uF; moved to F.Cu
- C54: renamed from C26; value 0.1uF -> 1uF
- C7: renamed from C13; value 0.1uF -> 1uF; moved to F.Cu
- H5, H6: footprint MountingHole:MountingHole_3.7mm_Pad -> MountingHole:MountingHole_3.7mm_Pad_TopOnly; moved to F.Cu
- J2: moved to F.Cu
- J4: renamed from J3; footprint Connector_PinHeader_2.54mm:PinHeader_1x04_P2.54mm_Vertical -> Connector_PinHeader_2.54mm:PinHeader_1x04_P2.54mm_Vertical_SMD_Pin1Left
- R1: renamed from R8; footprint Resistor_SMD:R_0603_1608Metric_Pad0.98x0.95mm_HandSolder -> Resistor_SMD:R_0402_1005Metric
- R10: renamed from R16; moved to F.Cu
- R11: renamed from R17; moved to F.Cu
- R12: renamed from R18; moved to F.Cu
- R15: value 10k -> 100k
- R2: renamed from R1; moved to F.Cu
- R22: renamed from R25; value 17k -> 40.2k
- R23: renamed from R26; value 100k -> 75k
- R3: renamed from R2; moved to F.Cu
- R4: renamed from R9; footprint Resistor_SMD:R_0603_1608Metric_Pad0.98x0.95mm_HandSolder -> Resistor_SMD:R_0402_1005Metric
- R7: renamed from R5; moved to F.Cu
- R8: renamed from R6; moved to F.Cu
- R9: renamed from R7; moved to F.Cu
- TP10, TP11: footprint TestPoint:TestPoint_THTPad_D2.0mm_Drill1.0mm -> TestPoint:TestPoint_Keystone_5000-5004_Miniature; moved to B.Cu
- TP4: footprint TestPoint:TestPoint_Pad_D1.0mm -> TestPoint:TestPoint_Keystone_5000-5004_Miniature
- TP9: renamed from TP6; footprint TestPoint:TestPoint_Pad_D1.0mm -> TestPoint:TestPoint_Keystone_5000-5004_Miniature; moved to B.Cu
- U1: value TVS2200DRV -> SN74LVC1G11; footprint Package_SON:WSON-6-1EP_2x2mm_P0.65mm_EP1x1.6mm -> Package_SON:Texas_USON-6_1x1.45mm_P0.5mm_SMD
- U13: renamed from U11; moved to F.Cu
- U4: value 74LVC1G07SE-7 -> 74LVC1G07; footprint Package_TO_SOT_SMD:SOT-353_SC-70-5 -> Package_SON:Texas_USON-6_1x1.45mm_P0.5mm_SMD
- U6: renamed from U5; moved to F.Cu
- moved TP4 98.4 mm to (144.5, 83.7), turned to 180 degrees
- moved TP11 72.5 mm to (149.5, 48.0), turned to 180 degrees
- moved TP2 69.6 mm to (158.9, 35.9), turned to 90 degrees
- moved R36 63.8 mm to (158.1, 34.4), turned to 180 degrees
- moved C54 63.5 mm to (157.7, 33.0), turned to 90 degrees
- moved R10 60.7 mm to (163.9, 78.1), turned to -90 degrees
- moved C20 58.8 mm to (162.8, 49.2), turned to 180 degrees
- moved R9 58.5 mm to (162.6, 78.1)
- moved U14 58.2 mm to (154.0, 33.4), turned to 0 degrees
- moved C22 57.8 mm to (162.8, 53.9), turned to 180 degrees
- moved C19 57.7 mm to (162.8, 51.6), turned to 180 degrees
- moved U6 57.3 mm to (162.0, 73.4)
- moved R8 55.9 mm to (161.3, 78.1)
- moved TP10 55.4 mm to (110.8, 42.9), turned to 180 degrees
- moved R11 53.6 mm to (163.9, 68.1)
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- renumbered C14 to C10, C15 to C11, C3 to C12, C4 to C13, C25 to C14, C5 to C15, C6 to C17, C31 to C19, C32 to C20, C37 to C21, C36 to C23, C39 to C24, C40 to C25, C38 to C26, C41 to C27, C16 to C28, C17 to C29, C18 to C30, C23 to C31, C44 to C32, C45 to C33, C7 to C34, C46 to C35, C24 to C36, C47 to C37, C48 to C38, C19 to C46, C20 to C47, C21 to C48, C22 to C49, C27 to C50, C28 to C51, C1 to C8, C2 to C9, J4 to J1, J1 to J3, L2 to L1, L3 to L2, R3 to R13, R4 to R14, R19 to R16, R20 to R17, R21 to R18, R22 to R19, R23 to R20, R24 to R21, R27 to R24, R28 to R25, R10 to R26, R29 to R27, R11 to R28, R12 to R29, R31 to R30, R32 to R31, R33 to R32, R30 to R36, TP2 to TP12, TP5 to TP14, TP1 to TP2, TP3 to TP8, U8 to U11, U12 to U14, U13 to U16, U6 to U8, U7 to U9
Connections:
- net Net-(J1-PadA4) renamed /Power/VIN
- net Net-(R3-Pad2) renamed /Power/CURRENT_SENSE_P
- net Net-(R3-Pad3) renamed /Power/CURRENT_SENSE_N
- J1 pad 10: /CM4 GPIO/TRD3_N -> /CM4 GPIO/TRD3_P
- J1 pad 3: /CM4 GPIO/TRD1_P -> /CM4 GPIO/TRD1_N
- J1 pad 4: /CM4 GPIO/TRD1_N -> /CM4 GPIO/TRD1_P
- J1 pad 9: /CM4 GPIO/TRD3_P -> /CM4 GPIO/TRD3_N
- J2 pad 10: unconnected-(J2-Pad10) -> Net-(J2-DAS/~{DSS}/~{LED1})
- J2 pad 50: /CM4 Highspeed/PCIE_nRST -> Net-(J2-~{PERST})
- J2 pad 52: /CM4 Highspeed/PCIE_CLK_nREQ -> Net-(J2-~{CLKREQ})
- Module1 pad 110: /CM4 Highspeed/PCIE_CLK_P -> /CM4 Highspeed/PCIE_CLK_N
- Module1 pad 112: /CM4 Highspeed/PCIE_CLK_N -> /CM4 Highspeed/PCIE_CLK_P
- Module1 pad 116: /CM4 Highspeed/PCIE_RX_P -> /CM4 Highspeed/PCIE_RX_N
- Module1 pad 118: /CM4 Highspeed/PCIE_RX_N -> /CM4 Highspeed/PCIE_RX_P
- Module1 pad 122: /CM4 Highspeed/PCIE_TX_P -> /CM4 Highspeed/PCIE_TX_N
- Module1 pad 124: /CM4 Highspeed/PCIE_TX_N -> /CM4 Highspeed/PCIE_TX_P
- Module1 pad 20: unconnected-(Module1-Pad20) -> /CM4 GPIO/EEPROM_nWP
- Module1 pad 28: unconnected-(Module1-Pad28) -> /CM4 GPIO/UART.RX
- Module1 pad 29: /CM4 GPIO/UART_WIRELESS_CTS -> unconnected-(Module1A-GPIO16-Pad29)
- Module1 pad 30: unconnected-(Module1-Pad30) -> /CM4 GPIO/Wireless.SWDIO
- Module1 pad 31: unconnected-(Module1-Pad31) -> /CM4 GPIO/UART.TX
- Module1 pad 35: unconnected-(Module1-Pad35) -> /CM4 GPIO/ID_SC
- Module1 pad 36: unconnected-(Module1-Pad36) -> /CM4 GPIO/ID_SD
- Module1 pad 37: unconnected-(Module1-Pad37) -> /CM4 GPIO/Wireless.SWCLK
- Module1 pad 38: /CM4 GPIO/SPI0_SCLK -> /CM4 GPIO/Wireless.RTS
- Module1 pad 39: /CM4 GPIO/SPI0_CE0 -> /CM4 GPIO/Wireless.TXD
- Module1 pad 40: /CM4 GPIO/SPI0_MISO -> /CM4 GPIO/Wireless.RXD
- Module1 pad 41: unconnected-(Module1-Pad41) -> /CM4 GPIO/Wireless.~{RESET}
- Module1 pad 44: /CM4 GPIO/SPI0_MOSI -> /CM4 GPIO/Wireless.CTS
- Module1 pad 45: unconnected-(Module1-Pad45) -> /CM4 GPIO/Wireless.~{BOOT}
- Module1 pad 46: unconnected-(Module1-Pad46) -> /CM4 GPIO/I2C.SDA
- Module1 pad 47: unconnected-(Module1-Pad47) -> /CM4 GPIO/I2C.SCL
- Module1 pad 50: /CM4 GPIO/UART_WIRELESS_RTS -> unconnected-(Module1A-GPIO17-Pad50)
- Module1 pad 51: /CM4 GPIO/UART_WIRELESS_RX -> unconnected-(Module1A-GPIO15-Pad51)
- Module1 pad 55: /CM4 GPIO/UART_WIRELESS_TX -> unconnected-(Module1A-GPIO14-Pad55)
- Module1 pad 82: /CM4 GPIO/SPI0_CE1 -> unconnected-(Module1A-SDA0-Pad82)
- Module1 pad 88: unconnected-(Module1-Pad88) -> +1V8
- Module1 pad 89: unconnected-(Module1-Pad89) -> Net-(Module1A-WiFi_nDisable)
- Module1 pad 90: unconnected-(Module1-Pad90) -> +1V8
- Module1 pad 91: unconnected-(Module1-Pad91) -> Net-(Module1A-BT_nDisable)
- Module1 pad 92: unconnected-(Module1-Pad92) -> /CM4 GPIO/RUN_PG
- Module1 pad 99: unconnected-(Module1-Pad99) -> Net-(Module1A-Global_EN)
- R15 pad 2: Net-(R15-Pad2) -> /Power/~{PWRDN}
- R16 pad 2: /Power/PGOOD1 -> /CM4 GPIO/3V3_PG
- R18 pad 1: /Power/PGOOD2 -> /CM4 GPIO/5V_PG
- TP10 pad 1: /Power/I2C_SCL -> /CM4 GPIO/3V3_PG
- TP11 pad 1: /CM4 GPIO/SPI0_SCLK -> /CM4 GPIO/5V_PG
- TP4 pad 1: +3V3 -> /CM4 GPIO/UART.RX
- U1 pad 1: GND -> /CM4 GPIO/3V3_PG
- U1 pad 3: GND -> /CM4 GPIO/5V_PG
- U1 pad 4: VBUS -> Net-(Module1A-Global_EN)
- U1 pad 5: VBUS -> +5V
- U1 pad 6: VBUS -> Net-(SW1-Pad4)
- U10 pad 1: /Power/PGOOD2 -> /CM4 GPIO/5V_PG
- U10 pad 24: /Power/PGOOD1 -> /CM4 GPIO/3V3_PG
- U13 pad 1: /Power/I2C_SDA -> /Sensors/I2C.SDA
- U13 pad 2: /Power/I2C_SCL -> /Sensors/I2C.SCL
- U14 pad 1: /Power/I2C_SDA -> /Sensors/I2C.SDA
- U14 pad 2: /Power/I2C_SCL -> /Sensors/I2C.SCL
- U16 pad 10: /CM4 GPIO/UART_WIRELESS_TX -> /CM4 GPIO/Wireless.TXD
- U16 pad 17: /CM4 GPIO/UART_WIRELESS_RTS -> /CM4 GPIO/Wireless.RTS
- U16 pad 2: unconnected-(U13-Pad2) -> /Wireless/~{LED_WIRELESS}
- U16 pad 22: /CM4 GPIO/UART_WIRELESS_CTS -> /CM4 GPIO/Wireless.CTS
- U16 pad 27: /CM4 GPIO/nEXTRST -> /CM4 GPIO/Wireless.~{RESET}
- U16 pad 29: Net-(AE1-Pad1) -> /Wireless/RF.Antenna
- U16 pad 3: unconnected-(U13-Pad3) -> Net-(U16-PB00)
- U16 pad 5: unconnected-(U13-Pad5) -> /CM4 GPIO/Wireless.SWCLK
- U16 pad 6: unconnected-(U13-Pad6) -> /CM4 GPIO/Wireless.SWDIO
- U16 pad 7: unconnected-(U13-Pad7) -> /CM4 GPIO/Wireless.SWO
- U16 pad 9: /CM4 GPIO/UART_WIRELESS_RX -> /CM4 GPIO/Wireless.RXD
- U4 pad 1: (no net) -> unconnected-(U4-NC-Pad1)
- U4 pad 5: +3.3V -> unconnected-(U4-NC-Pad5)
- U8 pad 10: unconnected-(U6-Pad10) -> GND
- U8 pad 13: unconnected-(U6-Pad13) -> GND
- U8 pad 19: unconnected-(U6-Pad19) -> GND
- U8 pad 26: unconnected-(U6-Pad26) -> GND
- U8 pad 27: unconnected-(U6-Pad27) -> GND
- U8 pad 36: unconnected-(U6-Pad36) -> GND
- U8 pad 37: unconnected-(U6-Pad37) -> GND
- U8 pad 5: unconnected-(U6-Pad5) -> GND
- U8 pad 6: unconnected-(U6-Pad6) -> GND
- U8 pad 7: unconnected-(U6-Pad7) -> GND
- U8 pad 8: /Power/I2C_SDA -> /Power/I2C.SDA
- U8 pad 9: /Power/I2C_SCL -> /Power/I2C.SCL
- U9 pad 4: /Power/I2C_SCL -> /Power/I2C.SCL
- U9 pad 5: /Power/I2C_SDA -> /Power/I2C.SDA
Routing:
- net /Power/I2C_SCL: track 103.8 -> 0.00 mm, vias 2 -> 0
- net /Power/I2C_SDA: track 101.5 -> 0.00 mm, vias 2 -> 0
- net /CM4 GPIO/3V3_PG: track 0.00 -> 88.2 mm, vias 0 -> 4
- net /Wireless/~{LED_WIRELESS}: track 0.00 -> 57.4 mm, vias 0 -> 3
- net VUSB: track 82.7 -> 136.9 mm, vias 3 -> 2
- net GND: track 2.53 -> 54.4 mm, vias 205 -> 408
- net /CM4 GPIO/nEXTRST: track 116.1 -> 68.4 mm, vias 5 -> 3
- net /CM4 GPIO/nPWR_LED: track 26.0 -> 72.3 mm
- net /CM4 GPIO/SPI0_CE0: track 45.2 -> 0.00 mm, vias 2 -> 0
- net +3.3V: track 286.6 -> 241.4 mm, vias 31 -> 23
- net /CM4 GPIO/SPI0_SCLK: track 44.3 -> 0.00 mm, vias 2 -> 0
- net /CM4 GPIO/SPI0_MOSI: track 43.5 -> 0.00 mm, vias 2 -> 0
- net /CM4 GPIO/Wireless.~{RESET}: track 0.00 -> 43.4 mm, vias 0 -> 3
- net /CM4 GPIO/SPI0_MISO: track 43.3 -> 0.00 mm, vias 2 -> 0
- net /CM4 GPIO/nLED_Activity: track 41.0 -> 80.7 mm, vias 2 -> 4
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- added copper zone on In2.Cu, net +3V3
- added copper zone on F.Cu, net /Power/LDO_1V5
- added copper zone on F.Cu, net /Power/LDO_3V3
- added copper zone on F.Cu, net VUSB
- removed copper zone on In2.Cu, net (none)
- removed copper zone on B.Cu, net +3V3
- removed copper zone on In2.Cu, net /Power/VIN
Other:
- board size 87.3 x 55.1 mm -> 107 x 55.9 mm
- board text added: "+5V PG"
- board text added: "ACT"
- board text added: "M.2"
- board text added: "M.2 PG"
- board text added: "OFF"
- board text added: "ON"
- board text added: "PWR"
- board text added: "RF"
- board text added: "RUN_PG"
- board text added: "RX"
- board text added: "TX"
- board text added: "ToDo: 1. Schalter für USB Boot 2. Schalter für GLOBAL_EN 3. Pad für RUN_PG 4. Reflow beidseitig ermöglichen"
- board text added: "UART"
- board text added: "USB PWR EN"
- board text added: "~{EXTRST}"
- board text added: "~{OC_FAULT}"
- board text removed: "+3.3V (CM4)"
- board text removed: "Rev 2"
- board text removed: "SPI_CLK"
- board text removed: "SPI_CS"
- board text removed: "SPI_MISO"
- board text removed: "SPI_MOSI"
- board text removed: "VBUS"

Commit message: Rev 2
Parts:
- removed the C12 at (149.8, 50.5)
- removed the C13 at (149.8, 52.4)
- removed the H4 at (61.1, 33.5)
- added C5: 10nF, Capacitor_SMD:C_0402_1005Metric, F.Cu at (67.1, 25.0)
- added C6: 10nF, Capacitor_SMD:C_0402_1005Metric, F.Cu at (67.1, 28.3)
- added R20: 100k, Resistor_SMD:R_0402_1005Metric, F.Cu at (75.9, 18.9)
- added REF**: KiCad-Logo2_5mm_SilkScreen, Symbol:KiCad-Logo2_5mm_SilkScreen, F.Cu at (138.6, 72.6)
- added REF**: OSHW-Symbol_6.7x6mm_SilkScreen, Symbol:OSHW-Symbol_6.7x6mm_SilkScreen, F.Cu at (138.7, 80.1)
- added REF**: WEEE-Logo_4.2x6mm_SilkScreen, Symbol:WEEE-Logo_4.2x6mm_SilkScreen, B.Cu at (132.8, 90.2)
- added REF**: RoHS-Logo_6mm_SilkScreen, Symbol:RoHS-Logo_6mm_SilkScreen, B.Cu at (110.7, 90.4)
- added REF**: ESD-Logo_6.6x6mm_SilkScreen, Symbol:ESD-Logo_6.6x6mm_SilkScreen, B.Cu at (126.0, 90.4)
- added REF**: Symbol_GNU-Logo_SilkscreenTop, Symbol:Symbol_GNU-Logo_SilkscreenTop, B.Cu at (81.5, 86.0)
- C40: renamed from C1; footprint Capacitor_SMD:C_0402_1005Metric -> Capacitor_SMD:C_0603_1608Metric
- C43: renamed from C52; footprint Capacitor_SMD:C_1206_3216Metric -> Capacitor_SMD:C_0402_1005Metric; moved to F.Cu
- J4: renamed from J7; moved to F.Cu
- J7: renamed from J6; moved to F.Cu
- R21: renamed from R15; footprint Resistor_SMD:R_0402_1005Metric -> Resistor_SMD:R_0805_2012Metric
- R36: renamed from R40; moved to F.Cu
- R37: renamed from R39; moved to F.Cu
- R40: renamed from R38; moved to F.Cu
- SW1, U16: moved to F.Cu
- TP1: renamed from TP11; moved to F.Cu
- TP12: renamed from TP1; moved to F.Cu
- TP13: renamed from TP15; moved to F.Cu
- TP14: renamed from TP16; moved to F.Cu
- TP15: renamed from TP9; moved to F.Cu
- TP2: renamed from TP20; moved to F.Cu
- TP3: renamed from TP18; moved to F.Cu
- TP6: renamed from TP10; moved to F.Cu
- TP9: renamed from TP3; moved to F.Cu
- U11: renamed from U12; moved to F.Cu
- moved H2 118.0 mm to (59.4, 91.6)
- moved R39 110.2 mm to (157.0, 21.8), turned to 0 degrees
- moved J2 102.2 mm to (60.9, 40.0)
- moved J1 101.6 mm to (60.8, 26.6), turned to -90 degrees
- moved C1 100.2 mm to (65.4, 35.0)
- moved R16 100.2 mm to (69.3, 35.0)
- moved R5 100.2 mm to (65.5, 44.9)
- moved R8 100.2 mm to (68.0, 35.0)
- moved R9 100.2 mm to (68.0, 44.9)
- moved R17 100.2 mm to (69.3, 44.9)
- moved R7 100.2 mm to (66.7, 44.9)
- moved U1 100.2 mm to (67.4, 40.2)
- moved FID3 98.1 mm to (66.1, 92.1)
- moved J5 98.0 mm to (154.8, 30.7), turned to 90 degrees
- moved FID1 96.8 mm to (155.1, 18.8)
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- renumbered C7 to C1, C39 to C10, C31 to C11, C32 to C12, C28 to C13, C3 to C14, C55 to C15, C33 to C16, C25 to C17, C37 to C18, C10 to C19, C30 to C2, C11 to C20, C35 to C21, C17 to C22, C15 to C23, C21 to C24, C36 to C25, C34 to C27, C24 to C28, C22 to C29, C27 to C3, C19 to C30, C20 to C31, C23 to C32, C14 to C33, C54 to C34, C6 to C35, C18 to C36, C16 to C37, C5 to C38, C4 to C39, C29 to C4, C56 to C41, C53 to C42, C45 to C44, C49 to C45, C44 to C46, C51 to C47, C2 to C49, C43 to C50, C41 to C51, C47 to C52, C46 to C53, C50 to C54, C42 to C55, C40 to C56, C38 to C7, FID3 to FID2, FID2 to FID3, H3 to H2, H6 to H3, H5 to H4, H2 to H5, H1 to H6, J3 to J1, J4 to J2, J2 to J3, J1 to J5, J5 to J6, L2 to L1, L1 to L2, R25 to R10, R24 to R11, R22 to R12, R17 to R13, R21 to R14, R20 to R15, R11 to R16, R10 to R17, R14 to R18, R13 to R19, R4 to R2, R26 to R22, R19 to R24, R18 to R25, R16 to R26, R36 to R27, R34 to R28, R33 to R29, R6 to R3, R5 to R30, R28 to R31, R29 to R33, R30 to R34, R31 to R35, R2 to R38, R3 to R39, R37 to R4, R7 to R5, R27 to R6, R8 to R7, R12 to R8, TP4 to TP10, TP5 to TP11, TP2 to TP16, TP14 to TP4, TP13 to TP5, TP8 to TP7, TP12 to TP8, U6 to U1, U5 to U10, U13 to U12, U2 to U13, U3 to U14, U11 to U15, U4 to U2, U15 to U3, U7 to U4, U10 to U5, U9 to U6, U8 to U7, U14 to U8, U1 to U9
Connections:
- C8 pad 1: VBUS -> /Power/VIN
- C9 pad 1: VBUS -> /Power/VIN
- J5 pad 10: /CM4 GPIO/TRD3_P -> /CM4 GPIO/TRD3_N
- J5 pad 9: /CM4 GPIO/TRD3_N -> /CM4 GPIO/TRD3_P
- TP2 pad 1: /Sensors/I2C.SCL -> /CM4 GPIO/I2C.SCL
- TP3 pad 1: /Sensors/I2C.SDA -> /CM4 GPIO/I2C.SDA
- U12 pad 1: /Sensors/I2C.SDA -> /CM4 GPIO/I2C.SDA
- U12 pad 2: /Sensors/I2C.SCL -> /CM4 GPIO/I2C.SCL
- U13 pad 1: /CM4 GPIO/TRD3_P -> /CM4 GPIO/TRD3_N
- U13 pad 10: /CM4 GPIO/TRD3_P -> /CM4 GPIO/TRD3_N
- U13 pad 2: /CM4 GPIO/TRD3_N -> /CM4 GPIO/TRD3_P
- U13 pad 9: /CM4 GPIO/TRD3_N -> /CM4 GPIO/TRD3_P
- U6 pad 4: /Power/I2C.SCL -> /CM4 GPIO/I2C.SCL
- U6 pad 5: /Power/I2C.SDA -> /CM4 GPIO/I2C.SDA
- U7 pad 8: /Power/I2C.SDA -> /CM4 GPIO/I2C.SDA
- U7 pad 9: /Power/I2C.SCL -> /CM4 GPIO/I2C.SCL
- U8 pad 1: /Sensors/I2C.SDA -> /CM4 GPIO/I2C.SDA
- U8 pad 2: /Sensors/I2C.SCL -> /CM4 GPIO/I2C.SCL
Routing:
- net /CM4 GPIO/I2C.SCL: track 0.00 -> 182.5 mm, vias 0 -> 4
- net /CM4 GPIO/I2C.SDA: track 0.00 -> 177.7 mm, vias 0 -> 4
- net +3.3V: track 241.4 -> 381.5 mm, vias 23 -> 19
- net /Wireless/~{LED_WIRELESS}: track 57.4 -> 147.8 mm, vias 3 -> 4
- net +5V: track 31.9 -> 104.6 mm, vias 3 -> 12
- net /CM4 GPIO/Wireless.CTS: track 26.3 -> 85.3 mm, vias 1 -> 2
- net /CM4 GPIO/Wireless.~{BOOT}: track 28.2 -> 84.3 mm, vias 1 -> 2
- net Net-(J3-DAS/~{DSS}/~{LED1}): track 11.1 -> 66.6 mm, vias 0 -> 2
- net /CM4 GPIO/Wireless.~{RESET}: track 43.4 -> 96.9 mm, vias 3 -> 2
- net /CM4 GPIO/Wireless.RXD: track 23.8 -> 76.5 mm, vias 1 -> 2
- net /CM4 GPIO/Wireless.SWCLK: track 30.0 -> 82.5 mm, vias 1 -> 2
- net GND: track 54.4 -> 106.8 mm, vias 408 -> 721
- net /CM4 GPIO/Wireless.RTS: track 22.9 -> 75.1 mm, vias 1 -> 2
- net /CM4 GPIO/Wireless.TXD: track 26.7 -> 78.5 mm, vias 1 -> 2
- net /CM4 GPIO/Wireless.SWDIO: track 30.1 -> 78.1 mm, vias 1 -> 2
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- added copper zone on B.Cu, net +5V
- removed copper zone on F.Cu, net +3.3V
- removed copper zone on In2.Cu, net +3V3
Other:
- board size 107 x 55.9 mm -> 104.1 x 77.9 mm
- board text added: "I²C"
- board text added: "Rev 2"
- board text removed: "I2C_SCL"
- board text removed: "I2C_SDA"
