File: rpi-cm-ssd.kicad_sch (KiCad schematic)
At the start: 7 parts

Commit message: Prep Rev2
Other:
- sheet CM4 GPIO ports: added 3V3_PG, 5V_PG, SPI{MISO MOSI SCLK CE}, Wireless{UART SWD ~{RESET} ~{BOOT}}; removed SPI0_CE0, SPI0_CE1, SPI0_MISO, SPI0_MOSI, SPI0_SCLK, UART_WIRELESS_CTS, UART_WIRELESS_RTS, UART_WIRELESS_RX, UART_WIRELESS_TX
- sheet CM4 Highspeed ports: added 3V3_PG; removed none
- sheet Power ports: added 3V3_PG, 5V_PG; removed PGOOD1, PGOOD2
- sheet Sensors ports: added SPI{MISO MOSI SCLK CE}; removed SPI_MISO, SPI_MOSI, SPI_SCLK, ~{SPI_BRIDGE_CS}
- sheet Wireless ports: added Wireless{UART SWD ~{RESET} ~{BOOT}}; removed UART_WIRELESS_CTS, UART_WIRELESS_RTS, UART_WIRELESS_RX, UART_WIRELESS_TX
- title: (none) -> Custom Homeassistant Base

Commit message: Rev 2
Parts:
- removed H4: MountingHole, MountingHole:MountingHole_2.7mm_M2.5, symbol Mechanical:MountingHole
- renumbered FID3 to FID2, FID2 to FID3, H3 to H2, H2 to H5, H1 to H6
Other:
- sheet CM4 GPIO ports: added I2C{SDA SCL}, UART{TX RX}; removed SPI{MISO MOSI SCLK CE}
- sheet Power ports: added I2C{SDA SCL}; removed I2C_SCL, I2C_SDA
- sheet Sensors ports: added I2C{SDA SCL}; removed I2C_SCL, I2C_SDA, SPI{MISO MOSI SCLK CE}
Changed lines of the file:
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@@
+	)
+	(junction
+		(at 175.26 104.14)
+		(diameter 0)
+		(color 0 0 0 0)
 	)
 	(junction
@@
 	(wire
 		(pts
-			(xy 232.41 62.23) (xy 236.22 62.23)
-		)
-		(stroke
-			(width 0)
-			(type default)
-		)
-	)
-	(wire
-		(pts
 			(xy 170.18 90.17) (xy 107.95 90.17)
 		)
@@
 	(wire
 		(pts
-			(xy 236.22 107.95) (xy 229.87 107.95)
-		)
-		(stroke
-			(width 0)
-			(type default)
-		)
-	)
-	(wire
-		(pts
 			(xy 107.95 90.17) (xy 107.95 100.33)
 		)
@@
 	(wire
 		(pts
-			(xy 238.76 110.49) (xy 229.87 110.49)
-		)
-		(stroke
-			(width 0)
-			(type default)
-		)
-	)
-	(wire
-		(pts
-			(xy 232.41 59.69) (xy 238.76 59.69)
-		)
-		(stroke
-			(width 0)
-			(type default)
-		)
-	)
-	(wire
-		(pts
 			(xy 100.33 100.33) (xy 107.95 100.33)
 		)
@@
 		)
 	)
-	(wire
-		(pts
-			(xy 238.76 59.69) (xy 238.76 110.49)
+	(bus
+		(pts
+			(xy 156.21 114.3) (xy 175.26 114.3)
 		)
 		(stroke
@@
 		)
 	)
+	(bus
+		(pts
+			(xy 180.34 66.04) (xy 175.26 66.04)
+		)
+		(stroke
+			(width 0)
+			(type default)
+		)
+	)
 	(wire
 		(pts
@@
 		)
 	)
+	(bus
+		(pts
+			(xy 175.26 114.3) (xy 175.26 104.14)
+		)
+		(stroke
+			(width 0)
+			(type default)
+		)
+	)
 	(wire
 		(pts
@@
 	(wire
 		(pts
-			(xy 236.22 62.23) (xy 236.22 107.95)
-		)
-		(stroke
-			(width 0)
-			(type default)
-		)
-	)
-	(wire
-		(pts
 			(xy 100.33 101.6) (xy 100.33 100.33)
 		)
@@
 		)
 	)
+	(bus
+		(pts
+			(xy 175.26 104.14) (xy 180.34 104.14)
+		)
+		(stroke
+			(width 0)
+			(type default)
+		)
+	)
 	(wire
 		(pts
@@
 	(bus
 		(pts
-			(xy 156.21 123.19) (xy 180.34 123.19)
+			(xy 175.26 66.04) (xy 175.26 104.14)
 		)
 		(stroke
@@
 			(width 0)
 			(type default)
-		)
-	)
-	(symbol
-		(lib_id "Mechanical:MountingHole")
-		(at 252.73 154.94 0)
-		(unit 1)
-		(exclude_from_sim no)
-		(in_bom no)
-		(on_board yes)
-		(dnp no)
-		(fields_autoplaced yes)
-		(property "Reference" "H4"
-			(at 255.27 153.6699 0)
-			(effects
-				(font
-					(size 1.27 1.27)
-				)
-				(justify left)
-			)
-		)
-		(property "Value" "MountingHole"
-			(at 255.27 156.2099 0)
-			(effects
-				(font
-					(size 1.27 1.27)
-				)
-				(justify left)
-			)
-		)
-		(property "Footprint" "MountingHole:MountingHole_2.7mm_M2.5"
-			(at 252.73 154.94 0)
-			(effects
-				(font
-					(size 1.27 1.27)
-				)
-				(hide yes)
-			)
-		)
-		(property "Datasheet" "~"
-			(at 252.73 154.94 0)
-			(effects
-				(font
-					(size 1.27 1.27)
-				)
-				(hide yes)
-			)
-		)
-		(property "Description" ""
-			(at 252.73 154.94 0)
-			(effects
-				(font
-					(size 1.27 1.27)
-				)
-				(hide yes)
-			)
-		)
-		(property "MPN" "KFS2-M2.5"
-			(at 252.73 154.94 0)
-			(effects
-				(font
-					(size 1.27 1.27)
-				)
-				(hide yes)
-			)
-		)
-		(instances
-			(project "rpi-cm-ssd"
-				(path "/d596c5fc-bc79-4446-9328-b82e41a34e97"
-					(reference "H4")
-					(unit 1)
-				)
-			)
 		)
 	)
@@
 		(dnp no)
 		(fields_autoplaced yes)
-		(property "Reference" "FID3"
+		(property "Reference" "FID2"
 			(at 255.27 138.4299 90)
 			(effects
@@
 			(project "rpi-cm-ssd"
 				(path "/d596c5fc-bc79-4446-9328-b82e41a34e97"
-					(reference "FID3")
+					(reference "FID2")
 					(unit 1)
 				)
@@
 		(dnp no)
 		(fields_autoplaced yes)
-		(property "Reference" "H2"
+		(property "Reference" "H5"
 			(at 210.82 153.6699 0)
 			(effects
@@
 			(project "rpi-cm-ssd"
 				(path "/d596c5fc-bc79-4446-9328-b82e41a34e97"
-					(reference "H2")
+					(reference "H5")
 					(unit 1)
 				)
@@
 		(dnp no)
 		(fields_autoplaced yes)
-		(property "Reference" "H1"
+		(property "Reference" "H6"
 			(at 189.23 153.6699 0)
 			(effects
@@
 			(project "rpi-cm-ssd"
 				(path "/d596c5fc-bc79-4446-9328-b82e41a34e97"
-					(reference "H1")
+					(reference "H6")
 					(unit 1)
 				)
@@
 		(dnp no)
 		(fields_autoplaced yes)
-		(property "Reference" "H3"
+		(property "Reference" "H2"
 			(at 233.68 153.6699 0)
 			(effects
@@
 			(project "rpi-cm-ssd"
 				(path "/d596c5fc-bc79-4446-9328-b82e41a34e97"
-					(reference "H3")
+					(reference "H2")
 					(unit 1)
 				)
@@
 		(dnp no)
 		(fields_autoplaced yes)
-		(property "Reference" "FID2"
+		(property "Reference" "FID3"
 			(at 255.27 133.3499 0)
 			(effects
@@
 			(project "rpi-cm-ssd"
 				(path "/d596c5fc-bc79-4446-9328-b82e41a34e97"
-					(reference "FID2")
+					(reference "FID3")
 					(unit 1)
 				)
@@
 			)
 		)
-		(pin "I2C_SCL" output
-			(at 229.87 107.95 0)
-			(effects
-				(font
-					(size 1.27 1.27)
-				)
-				(justify right)
-			)
-		)
-		(pin "I2C_SDA" bidirectional
-			(at 229.87 110.49 0)
-			(effects
-				(font
-					(size 1.27 1.27)
-				)
-				(justify right)
-			)
-		)
-		(pin "SPI{MISO MOSI SCLK CE}" bidirectional
-			(at 180.34 123.19 180)
+		(pin "I2C{SDA SCL}" bidirectional
+			(at 180.34 104.14 180)
 			(effects
 				(font
@@
 			)
 		)
-		(pin "SPI{MISO MOSI SCLK CE}" bidirectional
-			(at 156.21 123.19 0)
+		(pin "UART{TX RX}" bidirectional
+			(at 110.49 104.14 180)
+			(effects
+				(font
+					(size 1.27 1.27)
+				)
+				(justify left)
+			)
+		)
+		(pin "I2C{SDA SCL}" bidirectional
+			(at 156.21 114.3 0)
 			(effects
 				(font
@@
 			)
 		)
-		(pin "I2C_SDA" bidirectional
-			(at 232.41 59.69 0)
-			(effects
-				(font
-					(size 1.27 1.27)
-				)
-				(justify right)
-			)
-		)
-		(pin "I2C_SCL" input
-			(at 232.41 62.23 0)
-			(effects
-				(font
-					(size 1.27 1.27)
-				)
-				(justify right)
-			)
-		)
 		(pin "~{PWRDN}" input
 			(at 180.34 54.61 180)
@@
 			(effects
 				(font
+					(size 1.27 1.27)
+				)
+				(justify left)
+			)
+		)
+		(pin "I2C{SDA SCL}" bidirectional
+			(at 180.34 66.04 180)
+			(effects
+				(font
