File: sensors.kicad_sch (KiCad schematic)
At the start: 16 parts, among them U11 TCN75AVUA, U12 TCN75AVUA, U9 SC18IS604PWJ

Commit message: Prep Rev2
Parts:
- removed C10: 0.1uF, Capacitor_SMD:C_0402_1005Metric, symbol Device:C
- removed R13, R14: 4.7k, Resistor_SMD:R_0402_1005Metric, symbol Device:R
- removed R15: 10k, Resistor_SMD:R_0402_1005Metric, symbol Device:R
- removed TP11, TP12, TP7, TP9: TestPoint, TestPoint:TestPoint_THTPad_D2.0mm_Drill1.0mm, symbol Connector:TestPoint
- removed U9: SC18IS604PWJ, SC18IS604:SOP65P640X110-16N, symbol SC18IS604PWJ:SC18IS604PWJ
- C53: renamed from C11; value 0.1uF -> 1uF
- C54: renamed from C26; value 0.1uF -> 1uF
- TP18: renamed from TP8; footprint TestPoint:TestPoint_THTPad_D2.0mm_Drill1.0mm -> TestPoint:TestPoint_Keystone_5000-5004_Miniature
- TP20: renamed from TP10; footprint TestPoint:TestPoint_THTPad_D2.0mm_Drill1.0mm -> TestPoint:TestPoint_Keystone_5000-5004_Miniature
- renumbered R30 to R36, U11 to U13, U12 to U14
Connections:
- net I2C_SCL renamed I2C.SCL
- net I2C_SDA renamed I2C.SDA
- no-connect marks 5 -> 0
Other:
- note removed: "SPI to I2C bridge"
- moved on the sheet: C53, C54, R36, TP18, TP20, U13, U14

Commit message: Rev 2
Parts:
- U12: renamed from U13; LCSC Part # (none) -> C144336
- U8: renamed from U14; LCSC Part # (none) -> C144336
- renumbered C54 to C34, C53 to C42, R36 to R27, TP20 to TP2, TP18 to TP3
Changed lines of the file:
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@@
 		(dnp no)
 		(fields_autoplaced yes)
-		(property "Reference" "U13"
+		(property "Reference" "U12"
 			(at 67.31 26.67 0)
 			(effects
@@
 			)
 		)
+		(property "LCSC Part #" "C144336"
+			(at 53.34 34.29 0)
+			(effects
+				(font
+					(size 1.27 1.27)
+				)
+				(hide yes)
+			)
+		)
 		(pin "1"
 		)
@@
 			(project "rpi-cm-ssd"
 				(path "/d596c5fc-bc79-4446-9328-b82e41a34e97/83b039bf-d58d-4d6c-91b1-411c751c0a4c"
-					(reference "U13")
+					(reference "U12")
 					(unit 1)
 				)
@@
 		(dnp no)
 		(fields_autoplaced yes)
-		(property "Reference" "TP20"
+		(property "Reference" "TP2"
 			(at 151.13 48.7679 0)
 			(effects
@@
 			(project "rpi-cm-ssd"
 				(path "/d596c5fc-bc79-4446-9328-b82e41a34e97/83b039bf-d58d-4d6c-91b1-411c751c0a4c"
-					(reference "TP20")
+					(reference "TP2")
 					(unit 1)
 				)
@@
 		(dnp no)
 		(fields_autoplaced yes)
-		(property "Reference" "C54"
+		(property "Reference" "C34"
 			(at 105.41 77.4699 0)
 			(effects
@@
 			(project "rpi-cm-ssd"
 				(path "/d596c5fc-bc79-4446-9328-b82e41a34e97/83b039bf-d58d-4d6c-91b1-411c751c0a4c"
-					(reference "C54")
+					(reference "C34")
 					(unit 1)
 				)
@@
 		(dnp no)
 		(fields_autoplaced yes)
-		(property "Reference" "C53"
+		(property "Reference" "C42"
 			(at 104.14 36.8299 0)
 			(effects
@@
 			(project "rpi-cm-ssd"
 				(path "/d596c5fc-bc79-4446-9328-b82e41a34e97/83b039bf-d58d-4d6c-91b1-411c751c0a4c"
-					(reference "C53")
+					(reference "C42")
 					(unit 1)
 				)
@@
 		(dnp no)
 		(fields_autoplaced yes)
-		(property "Reference" "TP18"
+		(property "Reference" "TP3"
 			(at 135.89 48.7679 0)
 			(effects
@@
 			(project "rpi-cm-ssd"
 				(path "/d596c5fc-bc79-4446-9328-b82e41a34e97/83b039bf-d58d-4d6c-91b1-411c751c0a4c"
-					(reference "TP18")
+					(reference "TP3")
 					(unit 1)
 				)
@@
 		(dnp no)
 		(fields_autoplaced yes)
-		(property "Reference" "U14"
+		(property "Reference" "U8"
 			(at 68.58 67.31 0)
 			(effects
@@
 			)
 		)
+		(property "LCSC Part #" "C144336"
+			(at 54.61 74.93 0)
+			(effects
+				(font
+					(size 1.27 1.27)
+				)
+				(hide yes)
+			)
+		)
 		(pin "1"
 		)
@@
 			(project "rpi-cm-ssd"
 				(path "/d596c5fc-bc79-4446-9328-b82e41a34e97/83b039bf-d58d-4d6c-91b1-411c751c0a4c"
-					(reference "U14")
+					(reference "U8")
 					(unit 1)
 				)
@@
 		(dnp no)
 		(fields_autoplaced yes)
-		(property "Reference" "R36"
+		(property "Reference" "R27"
 			(at 95.25 77.4699 0)
 			(effects
@@
 			(project "rpi-cm-ssd"
 				(path "/d596c5fc-bc79-4446-9328-b82e41a34e97/83b039bf-d58d-4d6c-91b1-411c751c0a4c"
-					(reference "R36")
-					(unit 1)
-				)
+					(reference "R27")
+					(unit 1)
+				)
