File: usb.kicad_sch (KiCad schematic)
At the start: 16 parts, among them J5 690-008-221-904, U8 USB2512, Y1 24MHz

Commit message: Prep Rev2
Parts:
- added C40: 100uF, Capacitor_Tantalum_SMD:CP_EIA-3216-10_Kemet-I, symbol Device:C_Polarized
- added C42, C44, C45: 10uF, Capacitor_SMD:C_0603_1608Metric, symbol Device:C
- added TP15, TP16: TestPoint, TestPoint:TestPoint_Keystone_5000-5004_Miniature, symbol Connector:TestPoint
- C41: renamed from C8; value 15pF -> 15pF C0G
- C43: renamed from C9; value 15pF -> 15pF C0G
- renumbered C19 to C46, C20 to C47, C21 to C48, C22 to C49, C27 to C50, C28 to C51, R11 to R28, R12 to R29, R31 to R30, R32 to R31, R33 to R32, U8 to U11
Connections:
- net +3.3V: now also C44.2, C45.2
- net GND: now also C40.2, C42.1, C44.1, C45.1
- net USB_POWER_EN: now also TP16.1
- net VUSB: now also C40.1, C42.2
- net ~{OC_FAULT}: now also TP15.1

Commit message: Rev 2
Parts:
- U15: renamed from U11; LCSC Part # (none) -> C633332
- renumbered C45 to C44, C49 to C45, C44 to C46, C51 to C47, C43 to C50, C41 to C51, C47 to C52, C46 to C53, C50 to C54, C42 to C55, C40 to C56, J5 to J6, R28 to R31, R29 to R33, R30 to R34, R31 to R35, TP15 to TP13, TP16 to TP14
Changed lines of the file:
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@@
 		(dnp no)
 		(fields_autoplaced yes)
-		(property "Reference" "TP15"
+		(property "Reference" "TP13"
 			(at 193.04 25.9079 0)
 			(effects
@@
 			(project ""
 				(path "/d596c5fc-bc79-4446-9328-b82e41a34e97/8bad5741-37db-4b79-b533-af5ffd79bc37"
-					(reference "TP15")
+					(reference "TP13")
 					(unit 1)
 				)
@@
 		(dnp no)
 		(fields_autoplaced yes)
-		(property "Reference" "C41"
+		(property "Reference" "C51"
 			(at 44.45 81.2799 0)
 			(effects
@@
 			(project "rpi-cm-ssd"
 				(path "/d596c5fc-bc79-4446-9328-b82e41a34e97/8bad5741-37db-4b79-b533-af5ffd79bc37"
-					(reference "C41")
+					(reference "C51")
 					(unit 1)
 				)
@@
 		(on_board yes)
 		(dnp no)
-		(property "Reference" "C50"
+		(property "Reference" "C54"
 			(at 151.511 174.0916 0)
 			(effects
@@
 			(project "rpi-cm-ssd"
 				(path "/d596c5fc-bc79-4446-9328-b82e41a34e97/8bad5741-37db-4b79-b533-af5ffd79bc37"
-					(reference "C50")
+					(reference "C54")
 					(unit 1)
 				)
@@
 		(on_board yes)
 		(dnp no)
-		(property "Reference" "U11"
+		(property "Reference" "U15"
 			(at 96.52 38.1 0)
 			(effects
@@
 			)
 		)
+		(property "LCSC Part #" "C633332"
+			(at 120.65 74.93 0)
+			(effects
+				(font
+					(size 1.27 1.27)
+				)
+				(hide yes)
+			)
+		)
 		(pin "1"
 		)
@@
 			(project "rpi-cm-ssd"
 				(path "/d596c5fc-bc79-4446-9328-b82e41a34e97/8bad5741-37db-4b79-b533-af5ffd79bc37"
-					(reference "U11")
+					(reference "U15")
 					(unit 1)
 				)
@@
 		(on_board yes)
 		(dnp no)
-		(property "Reference" "R31"
+		(property "Reference" "R35"
 			(at 87.63 69.85 90)
 			(effects
@@
 			(project "rpi-cm-ssd"
 				(path "/d596c5fc-bc79-4446-9328-b82e41a34e97/8bad5741-37db-4b79-b533-af5ffd79bc37"
-					(reference "R31")
+					(reference "R35")
 					(unit 1)
 				)
@@
 		(on_board yes)
 		(dnp no)
-		(property "Reference" "C49"
+		(property "Reference" "C45"
 			(at 141.605 174.0916 0)
 			(effects
@@
 			(project "rpi-cm-ssd"
 				(path "/d596c5fc-bc79-4446-9328-b82e41a34e97/8bad5741-37db-4b79-b533-af5ffd79bc37"
-					(reference "C49")
+					(reference "C45")
 					(unit 1)
 				)
@@
 		(on_board yes)
 		(dnp no)
-		(property "Reference" "C45"
+		(property "Reference" "C44"
 			(at 99.06 173.9899 0)
 			(effects
@@
 			(project "rpi-cm-ssd"
 				(path "/d596c5fc-bc79-4446-9328-b82e41a34e97/8bad5741-37db-4b79-b533-af5ffd79bc37"
-					(reference "C45")
+					(reference "C44")
 					(unit 1)
 				)
@@
 		(dnp no)
 		(fields_autoplaced yes)
-		(property "Reference" "C43"
+		(property "Reference" "C50"
 			(at 53.34 90.1699 0)
 			(effects
@@
 			(project "rpi-cm-ssd"
 				(path "/d596c5fc-bc79-4446-9328-b82e41a34e97/8bad5741-37db-4b79-b533-af5ffd79bc37"
-					(reference "C43")
+					(reference "C50")
 					(unit 1)
 				)
@@
 		(on_board yes)
 		(dnp no)
-		(property "Reference" "C46"
+		(property "Reference" "C53"
 			(at 109.601 174.0916 0)
 			(effects
@@
 			(project "rpi-cm-ssd"
 				(path "/d596c5fc-bc79-4446-9328-b82e41a34e97/8bad5741-37db-4b79-b533-af5ffd79bc37"
-					(reference "C46")
+					(reference "C53")
 					(unit 1)
 				)
@@
 		(dnp no)
 		(fields_autoplaced yes)
-		(property "Reference" "TP16"
+		(property "Reference" "TP14"
 			(at 193.04 34.7979 0)
 			(effects
@@
 			(project ""
 				(path "/d596c5fc-bc79-4446-9328-b82e41a34e97/8bad5741-37db-4b79-b533-af5ffd79bc37"
-					(reference "TP16")
+					(reference "TP14")
 					(unit 1)
 				)
@@
 		(dnp no)
 		(fields_autoplaced yes)
-		(property "Reference" "C40"
+		(property "Reference" "C56"
 			(at 44.45 159.1309 0)
 			(effects
@@
 			(project "rpi-cm-ssd"
 				(path "/d596c5fc-bc79-4446-9328-b82e41a34e97/8bad5741-37db-4b79-b533-af5ffd79bc37"
-					(reference "C40")
+					(reference "C56")
 					(unit 1)
 				)
@@
 		(on_board yes)
 		(dnp no)
-		(property "Reference" "R28"
+		(property "Reference" "R31"
 			(at 61.595 111.125 90)
 			(effects
@@
 			(project "rpi-cm-ssd"
 				(path "/d596c5fc-bc79-4446-9328-b82e41a34e97/8bad5741-37db-4b79-b533-af5ffd79bc37"
-					(reference "R28")
+					(reference "R31")
 					(unit 1)
 				)
@@
 		(on_board yes)
 		(dnp no)
-		(property "Reference" "R30"
+		(property "Reference" "R34"
 			(at 76.835 111.125 90)
 			(effects
@@
 			(project "rpi-cm-ssd"
 				(path "/d596c5fc-bc79-4446-9328-b82e41a34e97/8bad5741-37db-4b79-b533-af5ffd79bc37"
-					(reference "R30")
+					(reference "R34")
 					(unit 1)
 				)
@@
 		(on_board yes)
 		(dnp no)
-		(property "Reference" "R29"
+		(property "Reference" "R33"
 			(at 69.215 111.125 90)
 			(effects
@@
 			(project "rpi-cm-ssd"
 				(path "/d596c5fc-bc79-4446-9328-b82e41a34e97/8bad5741-37db-4b79-b533-af5ffd79bc37"
-					(reference "R29")
+					(reference "R33")
 					(unit 1)
 				)
@@
 		(on_board yes)
 		(dnp no)
-		(property "Reference" "J5"
+		(property "Reference" "J6"
 			(at 219.075 110.49 0)
 			(effects
@@
 			(project "rpi-cm-ssd"
 				(path "/d596c5fc-bc79-4446-9328-b82e41a34e97/8bad5741-37db-4b79-b533-af5ffd79bc37"
-					(reference "J5")
+					(reference "J6")
 					(unit 1)
 				)
@@
 		(on_board yes)
 		(dnp no)
-		(property "Reference" "C47"
+		(property "Reference" "C52"
 			(at 121.031 174.0916 0)
 			(effects
@@
 			(project "rpi-cm-ssd"
 				(path "/d596c5fc-bc79-4446-9328-b82e41a34e97/8bad5741-37db-4b79-b533-af5ffd79bc37"
-					(reference "C47")
+					(reference "C52")
 					(unit 1)
 				)
@@
 		(on_board yes)
 		(dnp no)
-		(property "Reference" "C42"
+		(property "Reference" "C55"
 			(at 57.15 160.0199 0)
 			(effects
@@
 			(project "rpi-cm-ssd"
 				(path "/d596c5fc-bc79-4446-9328-b82e41a34e97/8bad5741-37db-4b79-b533-af5ffd79bc37"
-					(reference "C42")
+					(reference "C55")
 					(unit 1)
 				)
@@
 		(on_board yes)
 		(dnp no)
-		(property "Reference" "C44"
+		(property "Reference" "C46"
 			(at 87.63 173.9899 0)
 			(effects
@@
 			(project "rpi-cm-ssd"
 				(path "/d596c5fc-bc79-4446-9328-b82e41a34e97/8bad5741-37db-4b79-b533-af5ffd79bc37"
-					(reference "C44")
+					(reference "C46")
 					(unit 1)
 				)
@@
 		(on_board yes)
 		(dnp no)
-		(property "Reference" "C51"
+		(property "Reference" "C47"
 			(at 161.925 174.0916 0)
 			(effects
@@
 			(project "rpi-cm-ssd"
 				(path "/d596c5fc-bc79-4446-9328-b82e41a34e97/8bad5741-37db-4b79-b533-af5ffd79bc37"
-					(reference "C51")
+					(reference "C47")
 					(unit 1)
 				)
