File: wireless.kicad_sch (KiCad schematic)
At the start: 2 parts, among them U13 MGM210PB32JIA2

Commit message: Prep Rev2
Parts:
- removed AE1: A-4JA, A-4JA:A-4JA, symbol Device:Antenna_Shield
- added C55: 1uF, Capacitor_SMD:C_0402_1005Metric, symbol Device:C
- added D4: Blue 2.8V @ 5mA, LED_SMD:LED_0603_1608Metric, symbol Device:LED
- added J6: CONUFL001-SMD-T, Connector_Coaxial:U.FL_Hirose_U.FL-R-SMT-1_Vertical, symbol Connector:Conn_Coaxial
- added R37: 1k, Resistor_SMD:R_0402_1005Metric, symbol Device:R
- added R38: 1k, Resistor_SMD:R_0603_1608Metric, symbol Device:R
- added R39, R40: 10k, Resistor_SMD:R_0603_1608Metric, symbol Device:R
- added U15: SN74LVC1G07, Package_SON:Texas_USON-6_1x1.45mm_P0.5mm_SMD, symbol 74xGxx:74LVC1G07
- renumbered U13 to U16
Connections:
- net +3.3V: now also C55.1, D4.2 (A), R39.1, R40.1, U15.6 (VCC)
- net GND: now also C55.2, J6.2 (Ext), U15.3 (GND)
- net RF.Antenna: now reaches U16.29 (RF2G4_IO2)
- net RF.Antenna: now also J6.1 (In)
- net ~{LED_WIRELESS}: now reaches U16.2 (PB01)
- net ~{LED_WIRELESS}: now also U15.2
- net at U16.3 (PB00): now also R38.2, R39.2
- net Wireless.SWCLK: now reaches U16.5 (PA01)
- net Wireless.SWDIO: now reaches U16.6 (PA02)
- net Wireless.SWO: now reaches U16.7 (PA03)
- net UART_WIRELESS_CTS renamed Wireless.CTS
- net UART_WIRELESS_RTS renamed Wireless.RTS
- net UART_WIRELESS_RX renamed Wireless.RXD
- net UART_WIRELESS_TX renamed Wireless.TXD
- net nEXTRST renamed Wireless.~{RESET}
- net Wireless.~{RESET}: now also R40.2
- new net: R37.2, U15.4
- new net: D4.1 (K), R37.1
- new net Wireless.~{BOOT}: R38.1
Other:
- note added: "50Ω"
- note added: "Wireless activity LED"
- moved on the sheet: U16

Commit message: Rev 2
Parts:
- J7: renamed from J6; LCSC Part # (none) -> C22418213; MPN (none) -> CONUFL001-SMD-T
- U3: renamed from U15; LCSC Part # C2871155 -> C2675513; MPN SN74LVC1G07DPWR -> SN74LVC1G07DRY
- renumbered C55 to C15, R40 to R36, R39 to R37, R37 to R4, R38 to R40
Changed lines of the file:
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@@
 		(on_board yes)
 		(dnp no)
-		(property "Reference" "R38"
+		(property "Reference" "R40"
 			(at 68.58 31.242 90)
 			(effects
@@
 			(project ""
 				(path "/d596c5fc-bc79-4446-9328-b82e41a34e97/1676d548-828c-482e-aa18-249053c7cd27"
-					(reference "R38")
+					(reference "R40")
 					(unit 1)
 				)
@@
 		(dnp no)
 		(fields_autoplaced yes)
-		(property "Reference" "U15"
+		(property "Reference" "U3"
 			(at 56.134 107.442 0)
 			(effects
@@
 			)
 		)
-		(property "MPN" "SN74LVC1G07DPWR"
+		(property "MPN" "SN74LVC1G07DRY"
 			(at 51.816 121.666 0)
 			(effects
@@
 			)
 		)
-		(property "LCSC Part #" "C2871155"
+		(property "LCSC Part #" "C2675513"
 			(at 52.578 119.634 0)
 			(effects
@@
 			(project ""
 				(path "/d596c5fc-bc79-4446-9328-b82e41a34e97/1676d548-828c-482e-aa18-249053c7cd27"
-					(reference "U15")
+					(reference "U3")
 					(unit 1)
 				)
@@
 		(on_board yes)
 		(dnp no)
-		(property "Reference" "R39"
+		(property "Reference" "R37"
 			(at 76.454 30.48 0)
 			(effects
@@
 			(project ""
 				(path "/d596c5fc-bc79-4446-9328-b82e41a34e97/1676d548-828c-482e-aa18-249053c7cd27"
-					(reference "R39")
+					(reference "R37")
 					(unit 1)
 				)
@@
 		(on_board yes)
 		(dnp no)
-		(property "Reference" "R40"
+		(property "Reference" "R36"
 			(at 149.606 49.276 0)
 			(effects
@@
 			(project "rpi-cm-ssd"
 				(path "/d596c5fc-bc79-4446-9328-b82e41a34e97/1676d548-828c-482e-aa18-249053c7cd27"
-					(reference "R40")
+					(reference "R36")
 					(unit 1)
 				)
@@
 		(dnp no)
 		(fields_autoplaced yes)
-		(property "Reference" "J6"
+		(property "Reference" "J7"
 			(at 171.45 59.9831 0)
 			(effects
@@
 			)
 		)
+		(property "LCSC Part #" "C22418213"
+			(at 167.64 60.96 0)
+			(effects
+				(font
+					(size 1.27 1.27)
+				)
+				(hide yes)
+			)
+		)
+		(property "MPN" "CONUFL001-SMD-T"
+			(at 167.64 60.96 0)
+			(effects
+				(font
+					(size 1.27 1.27)
+				)
+				(hide yes)
+			)
+		)
 		(pin "1"
 		)
@@
 			(project ""
 				(path "/d596c5fc-bc79-4446-9328-b82e41a34e97/1676d548-828c-482e-aa18-249053c7cd27"
-					(reference "J6")
+					(reference "J7")
 					(unit 1)
 				)
@@
 		(dnp no)
 		(fields_autoplaced yes)
-		(property "Reference" "R37"
+		(property "Reference" "R4"
 			(at 68.58 111.7599 0)
 			(effects
@@
 			(project ""
 				(path "/d596c5fc-bc79-4446-9328-b82e41a34e97/1676d548-828c-482e-aa18-249053c7cd27"
-					(reference "R37")
+					(reference "R4")
 					(unit 1)
 				)
@@
 		(dnp no)
 		(fields_autoplaced yes)
-		(property "Reference" "C55"
+		(property "Reference" "C15"
 			(at 22.86 106.6799 0)
 			(effects
@@
 			(project ""
 				(path "/d596c5fc-bc79-4446-9328-b82e41a34e97/1676d548-828c-482e-aa18-249053c7cd27"
-					(reference "C55")
-					(unit 1)
-				)
+					(reference "C15")
+					(unit 1)
+				)
